File: src/hardware/fc/_autosave-drone.kicad_pcb (KiCad board)
At the start: 4 copper layers, 40 x 40 mm, 121 parts, among them J1 Conn_01x01, J10 Conn_01x01, J11 Conn_01x01, J12 Conn_01x01, J13 Conn_01x01, J14 Conn_01x01, J15 Conn_01x01, J16 Conn_01x01, J17 Conn_01x01, J18 Conn_01x01, J19 Conn_01x03, J2 Conn_01x08, J20 Conn_01x03, J21 Conn_01x03, J22 Conn_01x03, J23 Conn_01x01, J24 Conn_01x01, J25 Conn_01x01, J3 Conn_01x01, J4 Conn_01x01, J5 Conn_01x01, J6 Conn_01x01, J7 Conn_01x01, J8 Conn_01x01, J9 Conn_01x01, Q1 AO3400A, Q2 NPN, Q3 NPN, SW1 SW_Push, SW2 SW_Push, U10 LM66100DCKR, U2 TLV75533PDBVR, U3 W25Q128JVSIQTR, U4 STM32F405RGTx, U5 ICM-42688-P, U6 LP5907MFX-3.3/NOPB, U7 AT7456E, U8 MP4420HGJ-Z, U9 LM66100DCKR, X1 XL2EL89CSI-111YLC-27M, Y1 C115962

Commit message: new routing
Parts:
- moved J7 56.3 mm to (53.8, 35.5), turned to 180 degrees
- moved J6 56.0 mm to (51.5, 35.5), turned to 180 degrees
- moved J25 55.4 mm to (53.8, 32.8), turned to 180 degrees
- moved J4 51.0 mm to (51.5, 32.8), turned to 180 degrees
- moved J24 50.8 mm to (56.0, 32.8), turned to 180 degrees
- moved J11 49.0 mm to (56.0, 35.5), turned to 180 degrees
- moved J23 46.3 mm to (58.2, 32.8), turned to 180 degrees
- moved J10 44.3 mm to (58.2, 35.5), turned to 180 degrees
- moved J9 30.3 mm to (102.2, 67.8)
- moved J8 30.3 mm to (99.4, 67.8)
- moved J5 27.3 mm to (78.1, 39.3)
- moved J18 20.4 mm to (87.1, 39.3)
- moved J17 20.2 mm to (84.8, 39.3)
- moved J13 19.8 mm to (93.2, 27.0)
- moved J15 19.7 mm to (80.3, 39.3)
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Other:
- board text added: "+"
- board text added: "-"
- board text added: "5V"
- board text added: "9V"
- board text added: "9v"
- board text added: "GND"
- board text added: "RX"
- board text added: "TX"
- board text added: "VDD"
- board text added: "buzzer"
- board text added: "dji vtx"
- board text added: "power"
- board text added: "rx"
- board text added: "tx"
- board text added: "uart"
