File: src/hardware/fc/drone.kicad_sch (KiCad schematic)
At the start: 110 parts, among them J1 Conn_01x01, J10 Conn_01x01, J11 Conn_01x01, J12 Conn_01x01, J13 Conn_01x01, J14 Conn_01x01, J15 Conn_01x01, J16 Conn_01x01, J17 Conn_01x01, J18 Conn_01x01, J2 Conn_01x08, J3 Conn_01x01, J4 Conn_01x01, J5 Conn_01x01, J6 Conn_01x01, J7 Conn_01x01, J8 Conn_01x01, J9 Conn_01x01, Q1 AO3400A, Q2 NPN, Q3 NPN, SW1 SW_Push, SW2 SW_Push, U10 LM66100DCKR, U2 TLV75533PDBVR, U3 W25Q128JVSIQTR, U4 STM32F405RGTx, U5 ICM-42688-P, U6 LP5907MFX-3.3/NOPB, U7 AT7456E, U8 MP4420HGJ-Z, U9 LM66100DCKR, X1 XL2EL89CSI-111YLC-27M, Y1 C115962

Commit message: new routing
Parts:
- added J19, J20, J21, J22: Conn_01x03, footprint_lib:led_ring, symbol Connector_Generic:Conn_01x03
- added J23, J24, J25: Conn_01x01, footprint_lib:signal_pad, symbol Connector_Generic:Conn_01x01
- C19, C33, C34, C37: footprint Capacitor_SMD:C_1206_3216Metric -> Capacitor_SMD:C_0805_2012Metric; LCSC Part C1859 -> C45783
- C2, C27, C3: footprint Capacitor_SMD:C_0805_2012Metric -> Capacitor_SMD:C_0402_1005Metric; LCSC Part C49326713 -> C12530
- C39, C40, C8: footprint Capacitor_SMD:C_0805_2012Metric -> Capacitor_SMD:C_0402_1005Metric; LCSC Part C91185 -> C52923
- J1, J10, J11, J12, J13, J14, J15, J16, J17, J18, J3, J4, J5, J6, J7, J8, J9: footprint footprint-lib:signal_pad -> footprint_lib:signal_pad; now left out of the parts list
- R6: footprint Resistor_SMD:R_0603_1608Metric -> Resistor_SMD:R_0402_1005Metric; LCSC Part C23102 -> C25919
- R9: footprint Resistor_SMD:R_0603_1608Metric -> Resistor_SMD:R_0402_1005Metric; LCSC Part C21190 -> C11702
- TP1, TP2: footprint TestPoint:TestPoint_Pad_1.0x1.0mm -> footprint_lib:signal_pad
Connections:
- net +5V: now also J19.3 (Pin_3), J20.3 (Pin_3), J21.3 (Pin_3), J22.3 (Pin_3), J24.1 (Pin_1); no longer R3.1, R4.1, U10.3 (~{CE}), U9.5 (ST)
- net +9V: now also J23.1 (Pin_1)
- net GND: now also C1.1, C12.1, C4.1, C5.1, C6.1, J19.1 (Pin_1), J20.1 (Pin_1), J21.1 (Pin_1), J22.1 (Pin_1)
- net VDD: now also C1.2, C12.2, C4.2, C5.2, C6.2, U4.1 (VBAT), U4.19 (VDD), U4.32 (VDD), U4.48 (VDD), U4.64 (VDD), J25.1 (Pin_1); no longer C1.1, C12.1, C4.1, C5.1, C6.1
- net LED_4: now reaches U4.10 (PC2)
- net LED_4: now also J19.2 (Pin_2)
- net LED_1: now reaches U4.28 (PB2)
- net LED_1: now also J20.2 (Pin_2)
- net LED_2: now reaches U4.57 (PB5)
- net LED_2: now also J21.2 (Pin_2)
- net LED_3: now reaches U4.9 (PC1)
- net LED_3: now also J22.2 (Pin_2)
- new net: R3.1, R4.1, U10.3 (~{CE}), U9.5 (ST)
Other:
- note added: "additional pads"
- note added: "beatflight led strip"
